Commit message: Updates to Gazebo modle to more accurately model deepracer and the lidar

File: simulator/deepracer_sim/models/xacro/collision/deepracer_collision.xacro (robot description, xacro)
@@ -47,3 +47,15 @@
         <fdir1 value="1 0 0"/>
     </gazebo>
+    <!-- add bit mask -->
+    <!-- there is no collision for single and stereo camera, so no need to disable them -->
+    <!-- apply bit mask for four wheels and shell -->
+    <xacro:configure_collide_bitmask link_name="left_rear_wheel" bitmask="$(arg agent_bitmask)" />
+    <xacro:configure_collide_bitmask link_name="right_rear_wheel" bitmask="$(arg agent_bitmask)" />
+    <xacro:configure_collide_bitmask link_name="left_front_wheel" bitmask="$(arg agent_bitmask)" />
+    <xacro:configure_collide_bitmask link_name="right_front_wheel" bitmask="$(arg agent_bitmask)" />
+    <xacro:configure_collide_bitmask link_name="shell" bitmask="$(arg agent_bitmask)" />
+    <!-- apply bit mask for lidar if using lidar sensor -->
+    <xacro:if value="${'lidar' in sensor_type_val}">
+        <xacro:configure_collide_bitmask link_name="laser" bitmask="$(arg agent_bitmask)" />
+    </xacro:if>
 </robot>

File: simulator/deepracer_sim/models/xacro/deepracer/deepracer.xacro (robot description, xacro)
@@ -28,8 +28,8 @@
   <xacro:arg name="lidar_360_degree_max_angle" default="3.14" />
   <xacro:arg name="lidar_360_degree_min_range" default="0.15" />
-  <xacro:arg name="lidar_360_degree_max_range" default="10.0" />
-  <xacro:arg name="lidar_360_degree_range_resolution" default="0.01" />
+  <xacro:arg name="lidar_360_degree_max_range" default="12.0" />
+  <xacro:arg name="lidar_360_degree_range_resolution" default="0.12" />
   <xacro:arg name="lidar_360_degree_noise_mean" default="0.0" />
-  <xacro:arg name="lidar_360_degree_noise_stddev" default="0.01" />
+  <xacro:arg name="lidar_360_degree_noise_stddev" default="0.1" />
   <!-- convert sensor type from arg to property -->
   <xacro:property name="sensor_type_val" value="$(arg sensor_type)" />

File: simulator/deepracer_sim/models/xacro/sensor/deepracer_gazebo_lidar.xacro (robot description, xacro)
@@ -42,8 +42,8 @@
         <frameName>laser</frameName>
       </plugin>-->
-       <plugin name="rp_lidar" filename="libgazebo_ros_ray_sensor.so">
+       <plugin name="rplidar_ros" filename="libgazebo_ros_ray_sensor.so">
           <ros>
             <!-- <namespace>/laser</namespace> -->
-            <argument>~/out:=scan</argument>
+            <argument>~/out:=rplidar_ros/scan</argument>
           </ros>
           <output_type>sensor_msgs/LaserScan</output_type>

File: simulator/deepracer_sim/models/xacro/urdf/deepracer_stereo_cameras_and_lidar_urdf.xacro (robot description, xacro)
@@ -241,5 +241,5 @@
   <link name="laser">
     <inertial>
-      <origin xyz="0.006099 0.00028423 -0.012654" rpy="0 0 0" />
+      <origin xyz="0.0 0.0 0.0" rpy="0 0 0" />
       <mass value="1E-5" />
       <inertia ixx="1e-6" ixy="0" ixz="0" iyy="1e-6" iyz="0" izz="1e-6" />
@@ -261,5 +261,5 @@
   </link>
   <joint name="hokuyo_joint" type="fixed">
-    <origin xyz="0.02913 0 0.16145"  rpy="0 -0.0255 3.1416" />
+    <origin xyz="0.02913 0 0.16145"  rpy="0 0.02435 0" />
     <parent link="chassis" />
     <child link="laser" />
